File: hardware/tloc2/tloc2.kicad_sch (KiCad schematic)
At the start: 11 parts, among them M0 INMP441, M1 INMP441, M2 INMP441, M3 INMP441, U1 ESP32-WROOM-32

Commit message: before major refactor
Parts:
- added J1: PWR, symbol Connector:Conn_01x02_Socket
- C1, C2, C3, C4: value 150u -> 100n
- R1, R2: value 100k -> 44k
Connections:
- net 3V3_VDD: now also J1.2 (Pin_2)
- net GND: now also J1.1 (Pin_1)
Other:
- moved on the sheet: R1, R2
